File: dokumentation/kopplingsschema/gloria/gloria.sch (EAGLE design)
At the start: 27 parts, among them IC1 74LS125N

Commit message: Connected uninvoked pins.
Parts:
- ATMEGA1284P: value (none) -> SENSOR UNIT
- ATMEGA1284P1: value (none) -> DRIVE UNIT
- Q1, Q2: value (none) -> 16M
Connections:
- net GND: now also IC1P.GND, LINEENABLEMUX1P.VSS, LINEVALUEMUX1P.VSS
- net VCC: now also IC1P.VCC, LINEENABLEMUX1P.VDD, LINEVALUEMUX1P.VDD

Commit message: Added prototyping area.
Parts:
- added JP2: (no value), SparkFun-Connectors:M05NO_SILK
- added JP26, JP27, JP28, JP29, JP30, JP31, JP32, JP33, JP34, JP35, JP36: M11POGOPIN_HOLES_ONLY, SparkFun-Connectors:M11POGOPIN_HOLES_ONLY
- added JP3, JP4, JP5: (no value), SparkFun-Connectors:M06NO_SILK_FEMALE_PTH
Changed lines of the file:
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@@
 <grid distance="0.1" unitdist="inch" unit="inch" style="lines" multiple="1" display="no" altdistance="0.01" altunitdist="inch" altunit="inch"/>
 <layers>
-<layer number="1" name="Top" color="4" fill="1" visible="yes" active="no"/>
-<layer number="2" name="Route2" color="1" fill="3" visible="yes" active="no"/>
-<layer number="15" name="Route15" color="4" fill="6" visible="yes" active="no"/>
-<layer number="16" name="Bottom" color="1" fill="1" visible="yes" active="no"/>
-<layer number="17" name="Pads" color="2" fill="1" visible="yes" active="no"/>
-<layer number="18" name="Vias" color="2" fill="1" visible="yes" active="no"/>
-<layer number="19" name="Unrouted" color="6" fill="1" visible="yes" active="no"/>
-<layer number="20" name="Dimension" color="15" fill="1" visible="yes" active="no"/>
-<layer number="21" name="tPlace" color="7" fill="1" visible="yes" active="no"/>
-<layer number="22" name="bPlace" color="7" fill="1" visible="yes" active="no"/>
-<layer number="23" name="tOrigins" color="15" fill="1" visible="yes" active="no"/>
-<layer number="24" name="bOrigins" color="15" fill="1" visible="yes" active="no"/>
-<layer number="25" name="tNames" color="7" fill="1" visible="yes" active="no"/>
-<layer number="26" name="bNames" color="7" fill="1" visible="yes" active="no"/>
-<layer number="27" name="tValues" color="7" fill="1" visible="yes" active="no"/>
-<layer number="28" name="bValues" color="7" fill="1" visible="yes" active="no"/>
+<layer number="1" name="Top" color="4" fill="1" visible="no" active="no"/>
+<layer number="2" name="Route2" color="1" fill="3" visible="no" active="no"/>
+<layer number="15" name="Route15" color="4" fill="6" visible="no" active="no"/>
+<layer number="16" name="Bottom" color="1" fill="1" visible="no" active="no"/>
+<layer number="17" name="Pads" color="2" fill="1" visible="no" active="no"/>
+<layer number="18" name="Vias" color="2" fill="1" visible="no" active="no"/>
+<layer number="19" name="Unrouted" color="6" fill="1" visible="no" active="no"/>
+<layer number="20" name="Dimension" color="15" fill="1" visible="no" active="no"/>
+<layer number="21" name="tPlace" color="7" fill="1" visible="no" active="no"/>
+<layer number="22" name="bPlace" color="7" fill="1" visible="no" active="no"/>
+<layer number="23" name="tOrigins" color="15" fill="1" visible="no" active="no"/>
+<layer number="24" name="bOrigins" color="15" fill="1" visible="no" active="no"/>
+<layer number="25" name="tNames" color="7" fill="1" visible="no" active="no"/>
+<layer number="26" name="bNames" color="7" fill="1" visible="no" active="no"/>
+<layer number="27" name="tValues" color="7" fill="1" visible="no" active="no"/>
+<layer number="28" name="bValues" color="7" fill="1" visible="no" active="no"/>
 <layer number="29" name="tStop" color="7" fill="3" visible="no" active="no"/>
 <layer number="30" name="bStop" color="7" fill="6" visible="no" active="no"/>
@@
 <layer number="35" name="tGlue" color="7" fill="4" visible="no" active="no"/>
 <layer number="36" name="bGlue" color="7" fill="5" visible="no" active="no"/>
-<layer number="37" name="tTest" color="7" fill="1" visible="yes" active="no"/>
-<layer number="38" name="bTest" color="7" fill="1" visible="yes" active="no"/>
+<layer number="37" name="tTest" color="7" fill="1" visible="no" active="no"/>
+<layer number="38" name="bTest" color="7" fill="1" visible="no" active="no"/>
 <layer number="39" name="tKeepout" color="4" fill="11" visible="no" active="no"/>
 <layer number="40" name="bKeepout" color="1" fill="11" visible="no" active="no"/>
@@
 <layer number="44" name="Drills" color="7" fill="1" visible="no" active="no"/>
 <layer number="45" name="Holes" color="7" fill="1" visible="no" active="no"/>
-<layer number="46" name="Milling" color="3" fill="1" visible="yes" active="no"/>
-<layer number="47" name="Measures" color="7" fill="1" visible="yes" active="no"/>
-<layer number="48" name="Document" color="7" fill="1" visible="yes" active="no"/>
-<layer number="49" name="Reference" color="7" fill="1" visible="yes" active="no"/>
-<layer number="50" name="dxf" color="7" fill="1" visible="yes" active="no"/>
-<layer number="51" name="tDocu" color="7" fill="1" visible="yes" active="no"/>
-<layer number="52" name="bDocu" color="7" fill="1" visible="yes" active="no"/>
-<layer number="53" name="tGND_GNDA" color="7" fill="9" visible="yes" active="no"/>
-<layer number="54" name="bGND_GNDA" color="1" fill="9" visible="yes" active="no"/>
-<layer number="56" name="wert" color="7" fill="1" visible="yes" active="no"/>
-<layer number="57" name="tCAD" color="7" fill="1" visible="yes" active="no"/>
+<layer number="46" name="Milling" color="3" fill="1" visible="no" active="no"/>
+<layer number="47" name="Measures" color="7" fill="1" visible="no" active="no"/>
+<layer number="48" name="Document" color="7" fill="1" visible="no" active="no"/>
+<layer number="49" name="Reference" color="7" fill="1" visible="no" active="no"/>
+<layer number="50" name="dxf" color="7" fill="1" visible="no" active="no"/>
+<layer number="51" name="tDocu" color="7" fill="1" visible="no" active="no"/>
+<layer number="52" name="bDocu" color="7" fill="1" visible="no" active="no"/>
+<layer number="53" name="tGND_GNDA" color="7" fill="9" visible="no" active="no"/>
+<layer number="54" name="bGND_GNDA" color="1" fill="9" visible="no" active="no"/>
+<layer number="56" name="wert" color="7" fill="1" visible="no" active="no"/>
+<layer number="57" name="tCAD" color="7" fill="1" visible="no" active="no"/>
 <layer number="90" name="Modules" color="5" fill="1" visible="yes" active="yes"/>
 <layer number="91" name="Nets" color="2" fill="1" visible="yes" active="yes"/>
@@
 <part name="GND18" library="supply1" deviceset="GND" device=""/>
 <part name="P+11" library="supply1" deviceset="VCC" device=""/>
+<part name="JP26" library="SparkFun-Connectors" deviceset="M11" device="POGOPIN_HOLES_ONLY"/>
+<part name="JP27" library="SparkFun-Connectors" deviceset="M11" device="POGOPIN_HOLES_ONLY"/>
+<part name="JP28" library="SparkFun-Connectors" deviceset="M11" device="POGOPIN_HOLES_ONLY"/>
+<part name="JP29" library="SparkFun-Connectors" deviceset="M11" device="POGOPIN_HOLES_ONLY"/>
+<part name="JP30" library="SparkFun-Connectors" deviceset="M11" device="POGOPIN_HOLES_ONLY"/>
+<part name="JP31" library="SparkFun-Connectors" deviceset="M11" device="POGOPIN_HOLES_ONLY"/>
+<part name="JP32" library="SparkFun-Connectors" deviceset="M11" device="POGOPIN_HOLES_ONLY"/>
+<part name="JP33" library="SparkFun-Connectors" deviceset="M11" device="POGOPIN_HOLES_ONLY"/>
+<part name="JP34" library="SparkFun-Connectors" deviceset="M11" device="POGOPIN_HOLES_ONLY"/>
+<part name="JP35" library="SparkFun-Connectors" deviceset="M11" device="POGOPIN_HOLES_ONLY"/>
+<part name="JP36" library="SparkFun-Connectors" deviceset="M11" device="POGOPIN_HOLES_ONLY"/>
+<part name="JP3" library="SparkFun-Connectors" deviceset="M06" device="NO_SILK_FEMALE_PTH"/>
+<part name="JP4" library="SparkFun-Connectors" deviceset="M06" device="NO_SILK_FEMALE_PTH"/>
+<part name="JP5" library="SparkFun-Connectors" deviceset="M06" device="NO_SILK_FEMALE_PTH"/>
+<part name="JP2" library="SparkFun-Connectors" deviceset="M05" device="NO_SILK"/>
 </parts>
 <sheets>
@@
 <instance part="GND6" gate="1" x="40.64" y="-66.04"/>
 <instance part="P+9" gate="VCC" x="40.64" y="-45.72"/>
+<instance part="JP26" gate="G$1" x="91.44" y="-152.4"/>
+<instance part="JP27" gate="G$1" x="116.84" y="-152.4"/>
+<instance part="JP28" gate="G$1" x="142.24" y="-154.94"/>
+<instance part="JP29" gate="G$1" x="162.56" y="-154.94"/>
+<instance part="JP30" gate="G$1" x="187.96" y="-154.94"/>
+<instance part="JP31" gate="G$1" x="215.9" y="-157.48"/>
+<instance part="JP32" gate="G$1" x="236.22" y="-157.48"/>
+<instance part="JP33" gate="G$1" x="93.98" y="-195.58"/>
+<instance part="JP34" gate="G$1" x="129.54" y="-195.58"/>
+<instance part="JP35" gate="G$1" x="172.72" y="-198.12"/>
+<instance part="JP36" gate="G$1" x="210.82" y="-200.66"/>
+<instance part="JP3" gate="G$1" x="-86.36" y="-200.66"/>
+<instance part="JP4" gate="G$1" x="-55.88" y="-200.66"/>
+<instance part="JP5" gate="G$1" x="-60.96" y="-175.26"/>
+<instance part="JP2" gate="G$1" x="-73.66" y="-248.92"/>
 </instances>
 <busses>

Commit message: Rerouted board manually.
Parts:
- removed JP2: (no value), SparkFun-Connectors:M05NO_SILK
- removed JP3, JP4, JP5: (no value), SparkFun-Connectors:M06NO_SILK_FEMALE_PTH
- removed JP35, JP36: M11POGOPIN_HOLES_ONLY, SparkFun-Connectors:M11POGOPIN_HOLES_ONLY
- renumbered IC1 to TRISTATE
Changed lines of the file:
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@@
 </variantdefs>
 <classes>
-<class number="0" name="default" width="0" drill="0">
+<class number="0" name="signal" width="0.254" drill="0">
+<clearance class="0" value="0.254"/>
+</class>
+<class number="1" name="vcc" width="0.508" drill="0">
+<clearance class="1" value="0.254"/>
 </class>
 </classes>
@@
 <part name="GND2" library="supply1" deviceset="GND" device=""/>
 <part name="GND8" library="supply1" deviceset="GND" device=""/>
-<part name="IC1" library="74xx-eu" deviceset="74*125" device="N" technology="LS"/>
+<part name="TRISTATE" library="74xx-eu" deviceset="74*125" device="N" technology="LS"/>
 <part name="SENSOR_DISTANCE_1" library="con-molex" deviceset="22-23-2031" device=""/>
 <part name="SENSOR_DISTANCE_2" library="con-molex" deviceset="22-23-2031" device=""/>
@@
 <part name="JP33" library="SparkFun-Connectors" deviceset="M11" device="POGOPIN_HOLES_ONLY"/>
 <part name="JP34" library="SparkFun-Connectors" deviceset="M11" device="POGOPIN_HOLES_ONLY"/>
-<part name="JP35" library="SparkFun-Connectors" deviceset="M11" device="POGOPIN_HOLES_ONLY"/>
-<part name="JP36" library="SparkFun-Connectors" deviceset="M11" device="POGOPIN_HOLES_ONLY"/>
-<part name="JP3" library="SparkFun-Connectors" deviceset="M06" device="NO_SILK_FEMALE_PTH"/>
-<part name="JP4" library="SparkFun-Connectors" deviceset="M06" device="NO_SILK_FEMALE_PTH"/>
-<part name="JP5" library="SparkFun-Connectors" deviceset="M06" device="NO_SILK_FEMALE_PTH"/>
-<part name="JP2" library="SparkFun-Connectors" deviceset="M05" device="NO_SILK"/>
 </parts>
 <sheets>
@@
 <instance part="GND2" gate="1" x="-15.24" y="-2.54"/>
 <instance part="GND8" gate="1" x="83.82" y="15.24"/>
-<instance part="IC1" gate="A" x="58.42" y="12.7"/>
-<instance part="IC1" gate="B" x="71.12" y="25.4" rot="R90"/>
+<instance part="TRISTATE" gate="A" x="58.42" y="12.7"/>
+<instance part="TRISTATE" gate="B" x="71.12" y="25.4" rot="R90"/>
 <instance part="SERVO_UART" gate="-1" x="96.52" y="17.78"/>
 <instance part="SERVO_UART" gate="-2" x="96.52" y="15.24"/>
@@
 <instance part="C2" gate="G$1" x="-27.94" y="43.18" rot="R90"/>
 <instance part="C6" gate="G$1" x="-27.94" y="33.02" rot="R90"/>
-<instance part="IC1" gate="P" x="53.34" y="-27.94"/>
+<instance part="TRISTATE" gate="P" x="53.34" y="-27.94"/>
 <instance part="GND18" gate="1" x="53.34" y="-40.64"/>
 <instance part="P+11" gate="VCC" x="53.34" y="-15.24"/>
@@
 <wire x1="68.58" y1="12.7" x2="71.12" y2="12.7" width="0.1524" layer="91"/>
 <label x="68.58" y="10.16" size="1.778" layer="95"/>
-<pinref part="IC1" gate="A" pin="O"/>
-<pinref part="IC1" gate="B" pin="I"/>
+<pinref part="TRISTATE" gate="A" pin="O"/>
+<pinref part="TRISTATE" gate="B" pin="I"/>
 <pinref part="SERVO_UART" gate="-3" pin="S"/>
 <junction x="71.12" y="12.7"/>
@@
 </segment>
 <segment>
-<pinref part="IC1" gate="P" pin="VCC"/>
+<pinref part="TRISTATE" gate="P" pin="VCC"/>
 <pinref part="P+11" gate="VCC" pin="VCC"/>
 <wire x1="53.34" y1="-20.32" x2="53.34" y2="-17.78" width="0.1524" layer="91"/>
@@
 <segment>
 <pinref part="GND18" gate="1" pin="GND"/>
-<pinref part="IC1" gate="P" pin="GND"/>
+<pinref part="TRISTATE" gate="P" pin="GND"/>
 <wire x1="53.34" y1="-38.1" x2="53.34" y2="-35.56" width="0.1524" layer="91"/>
 </segment>
@@
 <net name="UART1TX" class="0">
 <segment>
-<pinref part="IC1" gate="A" pin="I"/>
+<pinref part="TRISTATE" gate="A" pin="I"/>
 <pinref part="ATMEGA1284P1" gate="G$1" pin="TXD1/INT1/PCINT27"/>
 <wire x1="48.26" y1="12.7" x2="33.02" y2="12.7" width="0.1524" layer="91"/>
@@
 <net name="UART1RX" class="0">
 <segment>
-<pinref part="IC1" gate="B" pin="O"/>
+<pinref part="TRISTATE" gate="B" pin="O"/>
 <wire x1="71.12" y1="35.56" x2="48.26" y2="35.56" width="0.1524" layer="91"/>
 <wire x1="48.26" y1="35.56" x2="48.26" y2="15.24" width="0.1524" layer="91"/>
@@
 <net name="STYR_UART_TX_E" class="0">
 <segment>
-<pinref part="IC1" gate="A" pin="OE"/>
+<pinref part="TRISTATE" gate="A" pin="OE"/>
 <wire x1="58.42" y1="20.32" x2="58.42" y2="63.5" width="0.1524" layer="91"/>
 <pinref part="ATMEGA1284P1" gate="G$1" pin="T1/CLK0/PCINT9"/>
@@
 <net name="STYR_UART_RX_E" class="0">
 <segment>
-<pinref part="IC1" gate="B" pin="OE"/>
+<pinref part="TRISTATE" gate="B" pin="OE"/>
 <wire x1="63.5" y1="25.4" x2="63.5" y2="66.04" width="0.1524" layer="91"/>
 <pinref part="ATMEGA1284P1" gate="G$1" pin="T0/XCK0/PCINT8"/>
@@
 <instance part="JP33" gate="G$1" x="93.98" y="-195.58"/>
 <instance part="JP34" gate="G$1" x="129.54" y="-195.58"/>
-<instance part="JP35" gate="G$1" x="172.72" y="-198.12"/>
-<instance part="JP36" gate="G$1" x="210.82" y="-200.66"/>
-<instance part="JP3" gate="G$1" x="-86.36" y="-200.66"/>
-<instance part="JP4" gate="G$1" x="-55.88" y="-200.66"/>
-<instance part="JP5" gate="G$1" x="-60.96" y="-175.26"/>
-<instance part="JP2" gate="G$1" x="-73.66" y="-248.92"/>
 </instances>
 <busses>

Commit message: updated kopplingsschema
Parts:
- removed JP26, JP27, JP28, JP29, JP30, JP31, JP32, JP33, JP34: M11POGOPIN_HOLES_ONLY, SparkFun-Connectors:M11POGOPIN_HOLES_ONLY
- added SENSOR_LINE1: 057-026-1, con-panduit:057-026-1
Connections:
- new net N$46: LINEENABLEMUX1A.X14, SENSOR_LINE1-25.S
- new net N$47: LINEVALUEMUX1A.X14, SENSOR_LINE1-24.S
- new net N$48: LINEENABLEMUX1A.X15, SENSOR_LINE1-3.S
- new net N$49: LINEVALUEMUX1A.X15, SENSOR_LINE1-6.S
Other:
- moved on the sheet: ATMEGA1284P, C11, C12, C9, JTAG_SEN-1, JTAG_SEN-10, JTAG_SEN-2, JTAG_SEN-3, JTAG_SEN-4, JTAG_SEN-5, JTAG_SEN-6, JTAG_SEN-7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
